File: kicad/ta101bc.kicad_sch (KiCad schematic)
At the start: 99 parts, among them J1 INPUT, J2 OUTPUT, J3 SUBSONIC, J4 POWER, J5 MM INPUT, J6 PHONO, J7 OUTPUT, J8 SUPPLY, Q1 BC549C, Q101 BC549C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

Commit message: MC resistor option, improve silkscreen
Other:
- note added: "use 120 with TA191 MC"
Changed lines of the file:
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@@
+		)
+	)
+	(text "use 120 with TA191 MC"
+		(exclude_from_sim no)
+		(at 135.89 91.694 0)
+		(effects
+			(font
+				(size 1.27 1.27)
+			)
+		)
+	)
+	(text "use 120 with TA191 MC"
+		(exclude_from_sim no)
+		(at 134.366 24.13 0)
+		(effects
+			(font
+				(size 1.27 1.27)
+			)
 		)
 	)
